File: probe06-ivy/probe06-ivy.kicad_pcb (KiCad board)
At the start: 2 copper layers, 81 x 81 mm, 108 parts, among them J1 USB_B_Micro, J2 Conn_Coaxial, Q1 S9014, SW1 SW_Push, U1 STM32F407VGTx, U2 MP1584EN, U3 AMS1117-3.3, U6 24LC32, Y1 8 MHz, Y2 32.768 KHz

Commit message: minor changes
Parts:
- moved D3 0.23 mm to (182.7, 96.9)
- moved R7 0.23 mm to (179.2, 96.9)
- moved D4 0.16 mm to (182.7, 94.4)
- moved R8 0.16 mm to (179.2, 94.5)
- moved D2 0.11 mm to (182.7, 99.4)
- moved R6 0.11 mm to (179.3, 99.4)
Routing:
- net GND: vias 70 -> 71
Changed lines of the file:
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@@
 	(footprint "LED_SMD:LED_0603_1608Metric"
 		(layer "F.Cu")
-		(at 182.7125 94.28 180)
+		(at 182.7075 94.44 180)
 		(descr "LED SMD 0603 (1608 Metric), square (rectangular) end terminal, IPC_7351 nominal, (Body size source: http://www.tortai-tech.com/upload/download/2011102023233369053.pdf), generated with kicad-footprint-generator")
 		(tags "LED")
@@
 	(footprint "Resistor_SMD:R_0603_1608Metric"
 		(layer "F.Cu")
-		(at 179.195 94.29 180)
+		(at 179.19 94.45 180)
 		(descr "Resistor SMD 0603 (1608 Metric), square (rectangular) end terminal, IPC_7351 nominal, (Body size source: IPC-SM-782 page 72, https://www.pcb-3d.com/wordpress/wp-content/uploads/ipc-sm-782a_amendment_1_and_2.pdf), generated with kicad-footprint-generator")
 		(tags "resistor")
@@
 	(footprint "LED_SMD:LED_0603_1608Metric"
 		(layer "F.Cu")
-		(at 182.7425 99.27 180)
+		(at 182.7375 99.38 180)
 		(descr "LED SMD 0603 (1608 Metric), square (rectangular) end terminal, IPC_7351 nominal, (Body size source: http://www.tortai-tech.com/upload/download/2011102023233369053.pdf), generated with kicad-footprint-generator")
 		(tags "LED")
@@
 		(fp_arc
 			(start 6.1679 9.656)
-			(mid 5.659554 9.609621)
+			(mid 5.659557 9.609613)
 			(end 5.168 9.472)
 			(stroke
@@
 	(footprint "Resistor_SMD:R_0603_1608Metric"
 		(layer "F.Cu")
-		(at 179.215 96.7 180)
+		(at 179.175 96.93 180)
 		(descr "Resistor SMD 0603 (1608 Metric), square (rectangular) end terminal, IPC_7351 nominal, (Body size source: IPC-SM-782 page 72, https://www.pcb-3d.com/wordpress/wp-content/uploads/ipc-sm-782a_amendment_1_and_2.pdf), generated with kicad-footprint-generator")
 		(tags "resistor")
@@
 	(footprint "Resistor_SMD:R_0603_1608Metric"
 		(layer "F.Cu")
-		(at 179.265 99.27 180)
+		(at 179.26 99.38 180)
 		(descr "Resistor SMD 0603 (1608 Metric), square (rectangular) end terminal, IPC_7351 nominal, (Body size source: IPC-SM-782 page 72, https://www.pcb-3d.com/wordpress/wp-content/uploads/ipc-sm-782a_amendment_1_and_2.pdf), generated with kicad-footprint-generator")
 		(tags "resistor")
@@
 	(footprint "LED_SMD:LED_0603_1608Metric"
 		(layer "F.Cu")
-		(at 182.72 96.69 180)
+		(at 182.68 96.92 180)
 		(descr "LED SMD 0603 (1608 Metric), square (rectangular) end terminal, IPC_7351 nominal, (Body size source: http://www.tortai-tech.com/upload/download/2011102023233369053.pdf), generated with kicad-footprint-generator")
 		(tags "LED")
@@
 	)
 	(segment
+		(start 179.3 108.08)
+		(end 181.835 110.615)
+		(width 0.3)
+		(layer "F.Cu")
+		(net 2)
+	)
+	(segment
 		(start 174.23 101.65)
 		(end 174.23 103.24)
@@
 	)
 	(segment
-		(start 178.2 101.45)
-		(end 179.3 102.55)
-		(width 0.3)
-		(layer "F.Cu")
-		(net 2)
-	)
-	(segment
 		(start 145.605 104.665)
 		(end 143.845 104.665)
@@
 	)
 	(segment
+		(start 181.835 110.615)
+		(end 181.835 110.87)
+		(width 0.3)
+		(layer "F.Cu")
+		(net 2)
+	)
+	(segment
 		(start 166.835 87.17)
 		(end 166.95 87.17)
@@
 	)
 	(segment
-		(start 179.3 102.55)
-		(end 179.3 108.335)
+		(start 173.68 83.04)
+		(end 173.68 84.52)
 		(width 0.3)
 		(layer "F.Cu")
@@
 	)
 	(segment
-		(start 173.68 83.04)
-		(end 173.68 84.52)
+		(start 177.2 101.45)
+		(end 178.2 101.45)
 		(width 0.3)
 		(layer "F.Cu")
@@
 	)
 	(segment
+		(start 179.3 102.55)
+		(end 179.3 108.08)
+		(width 0.3)
+		(layer "F.Cu")
+		(net 2)
+	)
+	(segment
 		(start 170.4725 91.1425)
 		(end 170.4725 93.0325)
@@
 	)
 	(segment
-		(start 177.2 101.45)
-		(end 178.2 101.45)
-		(width 0.3)
-		(layer "F.Cu")
-		(net 2)
-	)
-	(segment
 		(start 176.91 88.895)
 		(end 175.6 88.895)
@@
 	)
 	(segment
+		(start 178.2 101.45)
+		(end 179.3 102.55)
+		(width 0.3)
+		(layer "F.Cu")
+		(net 2)
+	)
+	(segment
 		(start 145.52 91.69)
 		(end 145.52 92.49)
@@
 	)
 	(segment
-		(start 179.3 108.335)
-		(end 181.835 110.87)
-		(width 0.3)
-		(layer "F.Cu")
-		(net 2)
-	)
-	(segment
 		(start 146.21 104.59)
 		(end 146.52 104.28)
@@
 	)
 	(segment
-		(start 151.5 105.44)
-		(end 151.53 105.44)
-		(width 0.3)
-		(layer "B.Cu")
-		(net 2)
-	)
-	(segment
 		(start 147.095 105.105)
 		(end 147.095 104.265)
@@
 		(net 149)
 	)
+	(via
+		(at 140.48 92.74)
+		(size 0.6)
+		(drill 0.3)
+		(layers "F.Cu" "B.Cu")
+		(net 149)
+	)

Commit message: mboh
Parts:
- removed R22, R23: 330, Resistor_SMD:R_0603_1608Metric
- renumbered AS5600 to AS5600_Encoder1, H206 to Autogyro1, BNO055 to BNO2, LED_PWR to LED_PWR1, U-BLOX to U4, XBEE to U5, BMP280 to U7
Connections:
- BT1 pad Neg: GND -> (no net)
- BT1 pad Pos: +3V0 -> (no net)
- U4 pad 20: Net-(U4-TXD/SPI_MISO) -> RX3
- U4 pad 21: Net-(U4-RXD/SPI_MOSI) -> TX3
Routing:
- net TX3: track 25.7 -> 29.5 mm
- net RX3: track 31.2 -> 34.2 mm
- net Net-(U4-TXD/SPI_MISO): track 2.86 -> 0.00 mm
- net Net-(U4-RXD/SPI_MOSI): track 2.44 -> 0.00 mm
